Commit message: bringup done, lidar not working

File: src/trover_description/urdf/trover_description.urdf.xacro (robot description, xacro)
@@ -17,16 +17,20 @@
   <xacro:property name="chassis_mass" value="${total_mass - 4*wheel_mass}"/>
   <!-- Wheel placement -->
-  <xacro:property name="wheel_x_offset" value="${chassis_length/2 - 0.0381}"/> <!-- -1.5 inches from chassis end-->
+  <xacro:property name="wheel_x_offset" value="${chassis_length/2 - 0.0381}"/>
   <xacro:property name="wheel_y_offset" value="${chassis_width/2 + wheel_width/2}"/>
   <xacro:property name="wheel_z" value="${wheel_radius}"/>
   <!-- Sensor placement -->
-  <xacro:property name="imu_z"
-                  value="${wheel_z + ground_clearance + chassis_height/2}"/>
-  <xacro:property name="lidar_x"
-                  value="0.0635"/>
-  <xacro:property name="lidar_y"
-                  value="-0.0508"/>
-  <xacro:property name="lidar_z"
-                  value="${ground_clearance + chassis_height + 0.06985}"/>
+  <xacro:property name="lidar_x" value="0.0635"/>
+  <xacro:property name="lidar_y" value="-0.0508"/>
+  <xacro:property name="lidar_z" value="${ground_clearance + chassis_height + 0.06985}"/>
+  <!-- ===================== -->
+  <!-- BASE FOOTPRINT (dummy link for KDL) -->
+  <!-- ===================== -->
+  <link name="base_footprint"/>
+  <joint name="base_joint" type="fixed">
+    <parent link="base_footprint"/>
+    <child link="base_link"/>
+    <origin xyz="0 0 0" rpy="0 0 0"/>
+  </joint>
   <!-- ===================== -->
   <!-- CHASSIS -->
@@ -35,5 +39,5 @@
     <inertial>
       <mass value="${chassis_mass}"/>
-      <origin xyz="0 0 0"/>
+      <origin xyz="0 0 ${ground_clearance + chassis_height/2}"/>
       <inertia
         ixx="${(1/12.0)*chassis_mass*(chassis_width*chassis_width + chassis_height*chassis_height)}"
@@ -58,4 +62,7 @@
     </collision>
   </link>
+  <gazebo reference="base_link">
+    <material>Gazebo/DarkGrey</material>
+  </gazebo>
   <!-- ===================== -->
   <!-- WHEEL MACRO -->
@@ -94,47 +101,122 @@
       <axis xyz="0 1 0"/>
     </joint>
+    <gazebo reference="${name}">
+      <material>Gazebo/FlatBlack</material>
+      <mu1>1.2</mu1>
+      <mu2>1.2</mu2>
+    </gazebo>
   </xacro:macro>
   <!-- ===================== -->
   <!-- WHEELS -->
   <!-- ===================== -->
-  <!-- Rear wheels (actuated + encoders) -->
   <xacro:wheel name="rear_left_wheel"  x="-${wheel_x_offset}" y="${wheel_y_offset}"/>
   <xacro:wheel name="rear_right_wheel" x="-${wheel_x_offset}" y="-${wheel_y_offset}"/>
-  <!-- Front wheels (mechanically coupled) -->
-  <xacro:wheel name="front_left_wheel"  x="${wheel_x_offset}" y="${wheel_y_offset}"/>
-  <xacro:wheel name="front_right_wheel" x="${wheel_x_offset}" y="-${wheel_y_offset}"/>
-  <joint name="front_left_mimic" type="continuous">
+  <!-- Front wheels (mechanically coupled via mimic) -->
+  <link name="front_left_wheel">
+    <inertial>
+      <mass value="${wheel_mass}"/>
+      <origin xyz="0 0 0"/>
+      <inertia
+        ixx="${(1/12.0)*wheel_mass*(3*wheel_radius*wheel_radius + wheel_width*wheel_width)}"
+        iyy="${(1/12.0)*wheel_mass*(3*wheel_radius*wheel_radius + wheel_width*wheel_width)}"
+        izz="${0.5*wheel_mass*wheel_radius*wheel_radius}"
+        ixy="0" ixz="0" iyz="0"/>
+    </inertial>
+    <visual>
+      <origin rpy="1.5708 0 0"/>
+      <geometry>
+        <cylinder radius="${wheel_radius}" length="${wheel_width}"/>
+      </geometry>
+      <material name="Black">
+        <color rgba="0.15 0.15 0.15 1"/>
+      </material>
+    </visual>
+    <collision>
+      <origin rpy="1.5708 0 0"/>
+      <geometry>
+        <cylinder radius="${wheel_radius}" length="${wheel_width}"/>
+      </geometry>
+    </collision>
+  </link>
+  <joint name="front_left_wheel_joint" type="continuous">
     <parent link="base_link"/>
     <child link="front_left_wheel"/>
+    <origin xyz="${wheel_x_offset} ${wheel_y_offset} ${wheel_z}"/>
+    <axis xyz="0 1 0"/>
     <mimic joint="rear_left_wheel_joint"/>
   </joint>
-  <joint name="front_right_mimic" type="continuous">
+  <gazebo reference="front_left_wheel">
+    <material>Gazebo/FlatBlack</material>
+    <mu1>1.2</mu1>
+    <mu2>1.2</mu2>
+  </gazebo>
+  <link name="front_right_wheel">
+    <inertial>
+      <mass value="${wheel_mass}"/>
+      <origin xyz="0 0 0"/>
+      <inertia
+        ixx="${(1/12.0)*wheel_mass*(3*wheel_radius*wheel_radius + wheel_width*wheel_width)}"
+        iyy="${(1/12.0)*wheel_mass*(3*wheel_radius*wheel_radius + wheel_width*wheel_width)}"
+        izz="${0.5*wheel_mass*wheel_radius*wheel_radius}"
+        ixy="0" ixz="0" iyz="0"/>
+    </inertial>
+    <visual>
+      <origin rpy="1.5708 0 0"/>
+      <geometry>
+        <cylinder radius="${wheel_radius}" length="${wheel_width}"/>
+      </geometry>
+      <material name="Black">
+        <color rgba="0.15 0.15 0.15 1"/>
+      </material>
+    </visual>
+    <collision>
+      <origin rpy="1.5708 0 0"/>
+      <geometry>
+        <cylinder radius="${wheel_radius}" length="${wheel_width}"/>
+      </geometry>
+    </collision>
+  </link>
+  <joint name="front_right_wheel_joint" type="continuous">
     <parent link="base_link"/>
     <child link="front_right_wheel"/>
+    <origin xyz="${wheel_x_offset} -${wheel_y_offset} ${wheel_z}"/>
+    <axis xyz="0 1 0"/>
     <mimic joint="rear_right_wheel_joint"/>
   </joint>
+  <gazebo reference="front_right_wheel">
+    <material>Gazebo/FlatBlack</material>
+    <mu1>1.2</mu1>
+    <mu2>1.2</mu2>
+  </gazebo>
   <!-- ===================== -->
   <!-- IMU -->
   <!-- ===================== -->
-  <link name="imu_link">
-    <inertial>
-      <mass value="0.01"/>
-      <origin xyz="0 0 0"/>
-      <inertia ixx="1e-5" iyy="1e-5" izz="1e-5"
-               ixy="0" ixz="0" iyz="0"/>
-    </inertial>
-  </link>
+  <link name="imu_link"/>
   <joint name="imu_joint" type="fixed">
     <parent link="base_link"/>
     <child link="imu_link"/>
-    <origin xyz="0 0 ${ground_clearance + chassis_height/2}"/>
+    <origin xyz="0 0 ${ground_clearance + chassis_height/2}" rpy="0 0 0"/>
   </joint>
   <gazebo reference="imu_link">
     <sensor name="imu_sensor" type="imu">
       <always_on>true</always_on>
-      <update_rate>200</update_rate>
+      <update_rate>100</update_rate>
+      <imu>
+        <angular_velocity>
+          <x><noise type="gaussian"><mean>0.0</mean><stddev>2e-4</stddev></noise></x>
+          <y><noise type="gaussian"><mean>0.0</mean><stddev>2e-4</stddev></noise></y>
+          <z><noise type="gaussian"><mean>0.0</mean><stddev>2e-4</stddev></noise></z>
+        </angular_velocity>
+        <linear_acceleration>
+          <x><noise type="gaussian"><mean>0.0</mean><stddev>1.7e-2</stddev></noise></x>
+          <y><noise type="gaussian"><mean>0.0</mean><stddev>1.7e-2</stddev></noise></y>
+          <z><noise type="gaussian"><mean>0.0</mean><stddev>1.7e-2</stddev></noise></z>
+        </linear_acceleration>
+      </imu>
       <plugin name="imu_plugin" filename="libgazebo_ros_imu_sensor.so">
-        <topicName>imu/data</topicName>
-        <frameName>imu_link</frameName>
+        <ros>
+          <remapping>~/out:=imu/data</remapping>
+        </ros>
+        <frame_name>imu_link</frame_name>
       </plugin>
     </sensor>
@@ -145,6 +227,7 @@
   <link name="lidar_link">
     <visual>
-      <geometry>
-        <cylinder radius="0.033" length="0.0254"/>
+      <origin xyz="0 0 0" rpy="0 0 0"/>
+      <geometry>
+        <cylinder radius="0.04" length="0.04"/>
       </geometry>
       <material name="purple">
@@ -153,13 +236,13 @@
     </visual>
     <collision>
-      <geometry>
-        <cylinder radius="0.033" length="0.0254"/>
+      <origin xyz="0 0 0" rpy="0 0 0"/>
+      <geometry>
+        <cylinder radius="0.04" length="0.04"/>
       </geometry>
     </collision>
     <inertial>
-      <mass value="0.05"/>
-      <origin xyz="0 0 0"/>
-      <inertia ixx="1e-4" iyy="1e-4" izz="1e-4"
-               ixy="0" ixz="0" iyz="0"/>
+      <mass value="0.1"/>
+      <origin xyz="0 0 0" rpy="0 0 0"/>
+      <inertia ixx="1e-4" iyy="1e-4" izz="1e-4" ixy="0" ixz="0" iyz="0"/>
     </inertial>
   </link>
@@ -167,14 +250,17 @@
     <parent link="base_link"/>
     <child link="lidar_link"/>
-    <origin xyz="${-lidar_x} ${lidar_y} ${lidar_z}"/>
+    <origin xyz="${-lidar_x} ${lidar_y} ${lidar_z}" rpy="0 0 0"/>
   </joint>
   <gazebo reference="lidar_link">
+    <material>Gazebo/Purple</material>
     <sensor name="lidar" type="ray">
       <always_on>true</always_on>
-      <update_rate>10</update_rate>
+      <visualize>true</visualize>
+      <update_rate>5</update_rate>
       <ray>
         <scan>
           <horizontal>
-            <samples>720</samples>
+            <samples>360</samples>
+            <resolution>1.0</resolution>
             <min_angle>-3.14159</min_angle>
             <max_angle>3.14159</max_angle>
@@ -182,24 +268,56 @@
         </scan>
         <range>
-          <min>0.12</min>
-          <max>12.0</max>
+          <min>0.15</min>
+          <max>10.0</max>
+          <resolution>0.01</resolution>
         </range>
+        <noise>
+          <type>gaussian</type>
+          <mean>0.0</mean>
+          <stddev>0.01</stddev>
+        </noise>
       </ray>
-      <plugin name="lidar_plugin" filename="libgazebo_ros_ray_sensor.so">
-        <topicName>scan</topicName>
-        <frameName>lidar_link</frameName>
+      <plugin name="scan" filename="libgazebo_ros_ray_sensor.so">
+        <ros>
+          <remapping>~/out:=scan</remapping>
+        </ros>
+        <output_type>sensor_msgs/LaserScan</output_type>
+        <frame_name>lidar_link</frame_name>
       </plugin>
     </sensor>
   </gazebo>
   <!-- ===================== -->
-  <!-- GAZEBO FRICTION -->
-  <!-- ===================== -->
-  <gazebo reference="rear_left_wheel">
-    <mu1>1.2</mu1>
-    <mu2>1.2</mu2>
-  </gazebo>
-  <gazebo reference="rear_right_wheel">
-    <mu1>1.2</mu1>
-    <mu2>1.2</mu2>
+  <!-- DIFFERENTIAL DRIVE -->
+  <!-- ===================== -->
+  <gazebo>
+    <plugin name="diff_drive" filename="libgazebo_ros_diff_drive.so">
+      <left_joint>rear_left_wheel_joint</left_joint>
+      <right_joint>rear_right_wheel_joint</right_joint>
+      <wheel_separation>${2 * wheel_y_offset}</wheel_separation>
+      <wheel_diameter>${wheel_diameter}</wheel_diameter>
+      <max_wheel_torque>20</max_wheel_torque>
+      <max_wheel_acceleration>1.0</max_wheel_acceleration>
+      <command_topic>cmd_vel</command_topic>
+      <odometry_topic>odom</odometry_topic>
+      <odometry_frame>odom</odometry_frame>
+      <robot_base_frame>base_link</robot_base_frame>
+      <publish_odom>true</publish_odom>
+      <publish_odom_tf>true</publish_odom_tf>
+      <publish_wheel_tf>false</publish_wheel_tf>
+      <update_rate>100</update_rate>
+    </plugin>
+  </gazebo>
+  <!-- ===================== -->
+  <!-- JOINT STATE PUBLISHER -->
+  <!-- ===================== -->
+  <gazebo>
+    <plugin name="joint_state_publisher" filename="libgazebo_ros_joint_state_publisher.so">
+      <ros>
+        <remapping>~/out:=joint_states</remapping>
+      </ros>
+      <update_rate>50</update_rate>
+      <joint_name>rear_left_wheel_joint</joint_name>
+      <joint_name>rear_right_wheel_joint</joint_name>
+    </plugin>
   </gazebo>
 </robot>

Commit message: lidar working

File: src/trover_description/urdf/trover_description.urdf.xacro (robot description, xacro)
@@ -253,37 +253,38 @@
   </joint>
   <gazebo reference="lidar_link">
-    <material>Gazebo/Purple</material>
-    <sensor name="lidar" type="ray">
-      <always_on>true</always_on>
-      <visualize>true</visualize>
-      <update_rate>5</update_rate>
-      <ray>
-        <scan>
-          <horizontal>
-            <samples>360</samples>
-            <resolution>1.0</resolution>
-            <min_angle>-3.14159</min_angle>
-            <max_angle>3.14159</max_angle>
-          </horizontal>
-        </scan>
-        <range>
-          <min>0.15</min>
-          <max>10.0</max>
-          <resolution>0.01</resolution>
-        </range>
-        <noise>
-          <type>gaussian</type>
-          <mean>0.0</mean>
-          <stddev>0.01</stddev>
-        </noise>
-      </ray>
-      <plugin name="scan" filename="libgazebo_ros_ray_sensor.so">
-        <ros>
-          <remapping>~/out:=scan</remapping>
-        </ros>
-        <output_type>sensor_msgs/LaserScan</output_type>
-        <frame_name>lidar_link</frame_name>
-      </plugin>
-    </sensor>
+  <material>Gazebo/Purple</material>
+  <sensor name="lidar" type="ray">
+    <always_on>true</always_on>
+    <visualize>true</visualize>
+    <update_rate>5</update_rate>
+    <ray>
+      <scan>
+        <horizontal>
+          <samples>360</samples>
+          <resolution>1.0</resolution>
+          <min_angle>-3.14159</min_angle>
+          <max_angle>3.14159</max_angle>
+        </horizontal>
+      </scan>
+      <range>
+        <min>0.15</min>
+        <max>10.0</max>
+        <resolution>0.01</resolution>
+      </range>
+      <noise>
+        <type>gaussian</type>
+        <mean>0.0</mean>
+        <stddev>0.01</stddev>
+      </noise>
+    </ray>
+    <plugin name="scan" filename="libgazebo_ros_ray_sensor.so">
+      <ros>
+        <namespace>/</namespace>
+        <remapping>~/out:=scan</remapping>
+      </ros>
+      <output_type>sensor_msgs/LaserScan</output_type>
+      <frame_name>lidar_link</frame_name>
+    </plugin>
+  </sensor>
   </gazebo>
   <!-- ===================== -->

Commit message: ROBOT IS ALIVE

File: src/trover_description/urdf/trover_description.urdf.xacro (robot description, xacro)
@@ -24,13 +24,4 @@
   <xacro:property name="lidar_y" value="-0.0508"/>
   <xacro:property name="lidar_z" value="${ground_clearance + chassis_height + 0.06985}"/>
-  <!-- ===================== -->
-  <!-- BASE FOOTPRINT (dummy link for KDL) -->
-  <!-- ===================== -->
-  <link name="base_footprint"/>
-  <joint name="base_joint" type="fixed">
-    <parent link="base_footprint"/>
-    <child link="base_link"/>
-    <origin xyz="0 0 0" rpy="0 0 0"/>
-  </joint>
   <!-- ===================== -->
   <!-- CHASSIS -->
@@ -103,6 +94,6 @@
     <gazebo reference="${name}">
       <material>Gazebo/FlatBlack</material>
-      <mu1>1.2</mu1>
-      <mu2>1.2</mu2>
+      <mu1>1.0</mu1>
+      <mu2>1.0</mu2>
     </gazebo>
   </xacro:macro>
@@ -144,10 +135,9 @@
     <origin xyz="${wheel_x_offset} ${wheel_y_offset} ${wheel_z}"/>
     <axis xyz="0 1 0"/>
-    <mimic joint="rear_left_wheel_joint"/>
   </joint>
   <gazebo reference="front_left_wheel">
     <material>Gazebo/FlatBlack</material>
-    <mu1>1.2</mu1>
-    <mu2>1.2</mu2>
+    <mu1>0.001</mu1>
+    <mu2>0.001</mu2>
   </gazebo>
   <link name="front_right_wheel">
@@ -182,10 +172,9 @@
     <origin xyz="${wheel_x_offset} -${wheel_y_offset} ${wheel_z}"/>
     <axis xyz="0 1 0"/>
-    <mimic joint="rear_right_wheel_joint"/>
   </joint>
   <gazebo reference="front_right_wheel">
     <material>Gazebo/FlatBlack</material>
-    <mu1>1.2</mu1>
-    <mu2>1.2</mu2>
+    <mu1>0.001</mu1>
+    <mu2>0.001</mu2>
   </gazebo>
   <!-- ===================== -->
@@ -293,4 +282,5 @@
   <gazebo>
     <plugin name="diff_drive" filename="libgazebo_ros_diff_drive.so">
+      <!-- 2WD: rear wheel drive only -->
       <left_joint>rear_left_wheel_joint</left_joint>
       <right_joint>rear_right_wheel_joint</right_joint>
